File: board_ems/ems_mbed/ems_mbed.sch (EAGLE design)
At the start: 146 parts, among them IC1 SIM900, IC2 74HC595D, IC3 74HC595D, IC4 ADE7758RW, J5 POWER_JACKPTH, U2 W5500

Commit message: add dht, mq6, and mq7 sensors
Parts:
- removed STM-S2: SWITCH-MOMENTARY-2PTH, SparkFun-Electromechanical:SWITCH-MOMENTARY-2PTH
- removed U$3: TFT_LCD_2.2, TFT_LCD_2.2:TFT_LCD_2.2
- added DHT-R1, MQ6-R1, MQ7-R1: 10k, resistor:R-EU_R0603
- added PB-GND, PB-SWD-NRST: (no value), adafruit:PINHD-1X1CB
- added SENSOR-DHT: (no value), pinhead:PINHD-1X4
- added SENSOR-MQ6, SENSOR-MQ7: METHANE_SENSOR, SparkFun-Sensors:METHANE_SENSOR
- added U$4: TFT_LCD_2.2+F_CS, TFT_LCD_2.2:TFT_LCD_2.2+F_CS
Connections:
- new net DHT_DATA: DHT-R1.2, SENSOR-DHT.2, STM_CHIP.PA1
- new net F_CS: STM_CHIP.PB10, U$4.F_CS
- new net MQ6_DATA: SENSOR-MQ7.B1, STM_CHIP.PB0
- new net MQ7_DATA: SENSOR-MQ6.B1, STM_CHIP.PB1
- new net N$43: MQ7-R1.2, SENSOR-MQ7.B2
- new net N$9: MQ6-R1.2, SENSOR-MQ6.B2
- net +5V: now also SENSOR-MQ6.A1, SENSOR-MQ6.A2, SENSOR-MQ6.HA, SENSOR-MQ7.A1, SENSOR-MQ7.A2, SENSOR-MQ7.HA
- net DGND: now also MQ6-R1.1, MQ7-R1.1, PB-GND.1, SENSOR-DHT.4, SENSOR-MQ6.HB, SENSOR-MQ7.HB, U$4.LCD_GND; no longer STM-S2.2, U$3.LCD_GND
- net LCD_CS: now also U$4.LCD_CS; no longer U$3.LCD_CS
- net LCD_D/C: now also U$4.LCD_D/C; no longer U$3.LCD_D/C
- net LCD_LED: now also U$4.LCD_LED; no longer U$3.LCD_LED
- net LCD_MISO: now also U$4.LCD_MISO, U$4.SD_MISO; no longer U$3.LCD_MISO, U$3.SD_MISO
- net LCD_MOSI: now also U$4.LCD_MOSI, U$4.SD_MOSI; no longer U$3.LCD_MOSI, U$3.SD_MOSI
- net LCD_RESET: now also U$4.LCD_RESET; no longer U$3.LCD_RESET
- net LCD_SCK: now also U$4.LCD_SCK, U$4.SD_SCK; no longer U$3.LCD_SCK, U$3.SD_SCK
- net SD_CS: now also U$4.SD_CS; no longer U$3.SD_CS
- net SWD_NRST: now also PB-SWD-NRST.1; no longer STM-S2.1
- net VDD: now also DHT-R1.1, SENSOR-DHT.1, U$4.LCD_VCC; no longer U$3.LCD_VCC
Other:
- moved on the sheet: ADE-C5, ADE-C6, LCD-R1

Commit message: add grber, chg ems_mbed w/ corct ones, del oth file
Parts:
- removed DHT-R1, MQ6-R1, MQ7-R1: 10k, resistor:R-EU_R0603
- removed PB-GND, PB-SWD-NRST: (no value), adafruit:PINHD-1X1CB
- removed SENSOR-DHT: (no value), pinhead:PINHD-1X4
- removed SENSOR-MQ6, SENSOR-MQ7: METHANE_SENSOR, SparkFun-Sensors:METHANE_SENSOR
- removed U$4: TFT_LCD_2.2+F_CS, TFT_LCD_2.2:TFT_LCD_2.2+F_CS
- added STM-S2: SWITCH-MOMENTARY-2PTH, SparkFun-Electromechanical:SWITCH-MOMENTARY-2PTH
- added U$3: TFT_LCD_2.2, TFT_LCD_2.2:TFT_LCD_2.2
Connections:
- removed net DHT_DATA: DHT-R1.2, SENSOR-DHT.2, STM_CHIP.PA1
- removed net F_CS: STM_CHIP.PB10, U$4.F_CS
- removed net MQ6_DATA: SENSOR-MQ7.B1, STM_CHIP.PB0
- removed net MQ7_DATA: SENSOR-MQ6.B1, STM_CHIP.PB1
- removed net N$43: MQ7-R1.2, SENSOR-MQ7.B2
- removed net N$9: MQ6-R1.2, SENSOR-MQ6.B2
- net +5V: no longer SENSOR-MQ6.A1, SENSOR-MQ6.A2, SENSOR-MQ6.HA, SENSOR-MQ7.A1, SENSOR-MQ7.A2, SENSOR-MQ7.HA
- net DGND: now also STM-S2.2, U$3.LCD_GND; no longer MQ6-R1.1, MQ7-R1.1, PB-GND.1, SENSOR-DHT.4, SENSOR-MQ6.HB, SENSOR-MQ7.HB, U$4.LCD_GND
- net LCD_CS: now also U$3.LCD_CS; no longer U$4.LCD_CS
- net LCD_D/C: now also U$3.LCD_D/C; no longer U$4.LCD_D/C
- net LCD_LED: now also U$3.LCD_LED; no longer U$4.LCD_LED
- net LCD_MISO: now also U$3.LCD_MISO, U$3.SD_MISO; no longer U$4.LCD_MISO, U$4.SD_MISO
- net LCD_MOSI: now also U$3.LCD_MOSI, U$3.SD_MOSI; no longer U$4.LCD_MOSI, U$4.SD_MOSI
- net LCD_RESET: now also U$3.LCD_RESET; no longer U$4.LCD_RESET
- net LCD_SCK: now also U$3.LCD_SCK, U$3.SD_SCK; no longer U$4.LCD_SCK, U$4.SD_SCK
- net SD_CS: now also U$3.SD_CS; no longer U$4.SD_CS
- net SWD_NRST: now also STM-S2.1; no longer PB-SWD-NRST.1
- net VDD: now also U$3.LCD_VCC; no longer DHT-R1.1, SENSOR-DHT.1, U$4.LCD_VCC
Other:
- moved on the sheet: ADE-C5, ADE-C6, LCD-R1
