File: board_ems/eth_module/eth_module.sch (EAGLE design)
At the start: 46 parts, among them Q1 25MHz, U1 W5500, U2 ARDUINOR3-DIMENSION

Commit message: add eth_module
Parts:
- added C20: C10uF/16V, resistor:CPOL-EU153CLV-0605
- added J1: POWER_JACKPTH, SparkFun-Connectors:POWER_JACKPTH
- added L1, L2: (no value), resistor:L-EUL2012C
- added U$2: DCDCMODULE_SMALL, bontor:DCDCMODULE_SMALL
Connections:
- removed net 3V3_ARDU: U2.3V
- new net PWRIN: J1.PWR, U$2.VIN
- net 3V3A: now also L1.1
- net 3V3ARDU: now also U2.3V
- net 3V3D: now also L2.1
- net 3V3IN: now also C20.+, L1.2, L2.2
- net 3V3PS: now also U$2.VOUT
- net GND: now also C20.-, J1.GND, J1.GNDBREAK, U$2.GNDI, U$2.GNDO
- net MISO: now also U2.D12
- net MOSI: now also U2.D11
- net SCLK: now also U2.D13
- net SCSN: now also U2.A2
- net W5500_NRST: now also U2.D10
Changed lines of the file:
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@@
 <layer number="54" name="bGND_GNDA" color="1" fill="9" visible="no" active="no"/>
 <layer number="56" name="wert" color="7" fill="1" visible="no" active="no"/>
+<layer number="57" name="tCAD" color="7" fill="1" visible="no" active="no"/>
 <layer number="91" name="Nets" color="2" fill="1" visible="yes" active="yes"/>
 <layer number="92" name="Busses" color="1" fill="1" visible="yes" active="yes"/>
@@
 <layer number="97" name="Info" color="7" fill="1" visible="yes" active="yes"/>
 <layer number="98" name="Guide" color="6" fill="1" visible="yes" active="yes"/>
+<layer number="99" name="SpiceOrder" color="7" fill="1" visible="yes" active="yes"/>
 <layer number="100" name="Muster" color="7" fill="1" visible="yes" active="yes"/>
 <layer number="101" name="Patch_Top" color="12" fill="4" visible="yes" active="yes"/>
@@
 <layer number="111" name="MPL" color="7" fill="1" visible="yes" active="yes"/>
 <layer number="112" name="tSilk" color="7" fill="1" visible="yes" active="yes"/>
+<layer number="113" name="IDFDebug" color="4" fill="1" visible="yes" active="yes"/>
 <layer number="116" name="Patch_BOT" color="9" fill="4" visible="yes" active="yes"/>
 <layer number="121" name="sName" color="7" fill="1" visible="yes" active="yes"/>
@@
 <layer number="132" name="bAdjust" color="7" fill="1" visible="no" active="yes"/>
 <layer number="144" name="Drill_legend" color="7" fill="1" visible="yes" active="yes"/>
+<layer number="150" name="Notes" color="7" fill="1" visible="yes" active="yes"/>
 <layer number="151" name="HeatSink" color="7" fill="1" visible="yes" active="yes"/>
 <layer number="152" name="_bDocu" color="7" fill="1" visible="yes" active="yes"/>
+<layer number="153" name="FabDoc1" color="7" fill="1" visible="yes" active="yes"/>
+<layer number="154" name="FabDoc2" color="7" fill="1" visible="yes" active="yes"/>
+<layer number="155" name="FabDoc3" color="7" fill="1" visible="yes" active="yes"/>
 <layer number="199" name="Contour" color="7" fill="1" visible="yes" active="yes"/>
 <layer number="200" name="200bmp" color="1" fill="10" visible="yes" active="yes"/>
@@
 <part name="U2" library="adafruit" deviceset="ARDUINOR3" device="-DIMENSION"/>
 <part name="POWER_SEL" library="adafruit" deviceset="PINHD-1X3" device=""/>
+<part name="J1" library="SparkFun-Connectors" deviceset="POWER_JACK" device="PTH"/>
+<part name="U$2" library="bontor" deviceset="DCDCMODULE_SMALL" device=""/>
+<part name="C20" library="resistor" deviceset="CPOL-EU" device="153CLV-0605" value="C10uF/16V"/>
+<part name="L1" library="resistor" deviceset="L-EU" device="L2012C"/>
+<part name="L2" library="resistor" deviceset="L-EU" device="L2012C"/>
 </parts>
 <sheets>
@@
 <instance part="U2" gate="G$1" x="99.06" y="187.96" rot="R270"/>
 <instance part="POWER_SEL" gate="A" x="25.4" y="190.5" rot="R180"/>
+<instance part="J1" gate="G$1" x="-76.2" y="203.2"/>
+<instance part="U$2" gate="G$1" x="-20.32" y="208.28"/>
+<instance part="C20" gate="G$1" x="27.94" y="160.02"/>
+<instance part="L1" gate="G$1" x="35.56" y="165.1" rot="R270"/>
+<instance part="L2" gate="G$1" x="35.56" y="170.18" rot="R270"/>
 </instances>
 <busses>
@@
 <wire x1="142.24" y1="129.54" x2="147.32" y2="129.54" width="0.1524" layer="91"/>
 </segment>
+<segment>
+<pinref part="L1" gate="G$1" pin="1"/>
+<wire x1="40.64" y1="165.1" x2="43.18" y2="165.1" width="0.1524" layer="91"/>
+<label x="43.18" y="165.1" size="1.27" layer="95" xref="yes"/>
+</segment>
 </net>
 <net name="N$2" class="0">
@@
 <label x="66.04" y="185.42" size="1.27" layer="95" rot="R180" xref="yes"/>
 </segment>
+<segment>
+<pinref part="J1" gate="G$1" pin="GNDBREAK"/>
+<pinref part="J1" gate="G$1" pin="GND"/>
+<wire x1="-73.66" y1="208.28" x2="-73.66" y2="205.74" width="0.1524" layer="91"/>
+<wire x1="-73.66" y1="205.74" x2="-71.12" y2="205.74" width="0.1524" layer="91"/>
+<label x="-71.12" y="205.74" size="1.27" layer="95" xref="yes"/>
+</segment>
+<segment>
+<pinref part="U$2" gate="G$1" pin="GNDI"/>
+<wire x1="-55.88" y1="200.66" x2="-55.88" y2="198.12" width="0.1524" layer="91"/>
+<label x="-55.88" y="198.12" size="1.27" layer="95" rot="R180" xref="yes"/>
+</segment>
+<segment>
+<pinref part="U$2" gate="G$1" pin="GNDO"/>
+<wire x1="15.24" y1="200.66" x2="15.24" y2="198.12" width="0.1524" layer="91"/>
+<label x="15.24" y="198.12" size="1.27" layer="95" xref="yes"/>
+</segment>
+<segment>
+<pinref part="C20" gate="G$1" pin="-"/>
+<wire x1="27.94" y1="154.94" x2="27.94" y2="152.4" width="0.1524" layer="91"/>
+<label x="27.94" y="152.4" size="1.27" layer="95" xref="yes"/>
+</segment>
 </net>
 <net name="TXN" class="0">
@@
 <wire x1="193.04" y1="144.78" x2="190.5" y2="144.78" width="0.1524" layer="91"/>
 <label x="190.5" y="144.78" size="1.27" layer="95" rot="R180" xref="yes"/>
+</segment>
+<segment>
+<pinref part="L2" gate="G$1" pin="1"/>
+<wire x1="40.64" y1="170.18" x2="43.18" y2="170.18" width="0.1524" layer="91"/>
+<label x="43.18" y="170.18" size="1.27" layer="95" xref="yes"/>
 </segment>
 </net>
@@
 <wire x1="243.84" y1="109.22" x2="243.84" y2="106.68" width="0.1524" layer="91"/>
 </segment>
+<segment>
+<pinref part="U2" gate="G$1" pin="A2"/>
+<wire x1="68.58" y1="172.72" x2="66.04" y2="172.72" width="0.1524" layer="91"/>
+<label x="66.04" y="172.72" size="1.27" layer="95" rot="R180" xref="yes"/>
+</segment>
 </net>
 <net name="SCLK" class="0">
@@
 <label x="231.14" y="109.22" size="1.27" layer="95" xref="yes"/>
 </segment>
+<segment>
+<pinref part="U2" gate="G$1" pin="D13"/>
+<wire x1="129.54" y1="203.2" x2="132.08" y2="203.2" width="0.1524" layer="91"/>
+<label x="132.08" y="203.2" size="1.27" layer="95" xref="yes"/>
+</segment>
 </net>
 <net name="MISO" class="0">
@@
 <label x="231.14" y="111.76" size="1.27" layer="95" xref="yes"/>
 </segment>
+<segment>
+<pinref part="U2" gate="G$1" pin="D12"/>
+<wire x1="129.54" y1="200.66" x2="132.08" y2="200.66" width="0.1524" layer="91"/>
+<label x="132.08" y="200.66" size="1.27" layer="95" xref="yes"/>
+</segment>
 </net>
 <net name="MOSI" class="0">
@@
 <wire x1="228.6" y1="114.3" x2="231.14" y2="114.3" width="0.1524" layer="91"/>
 <label x="231.14" y="114.3" size="1.27" layer="95" xref="yes"/>
+</segment>
+<segment>
+<pinref part="U2" gate="G$1" pin="D11"/>
+<wire x1="129.54" y1="198.12" x2="132.08" y2="198.12" width="0.1524" layer="91"/>
+<label x="132.08" y="198.12" size="1.27" layer="95" xref="yes"/>
 </segment>
 </net>
@@
 <label x="215.9" y="132.08" size="1.27" layer="95" xref="yes"/>
 </segment>
+<segment>
+<pinref part="U2" gate="G$1" pin="D10"/>
+<wire x1="129.54" y1="195.58" x2="132.08" y2="195.58" width="0.1524" layer="91"/>
+<label x="132.08" y="195.58" size="1.27" layer="95" xref="yes"/>
+</segment>
 </net>
 <net name="N$13" class="0">
@@
 </segment>
 </net>
-<net name="3V3_ARDU" class="0">
+<net name="3V3IN" class="0">
+<segment>
+<pinref part="POWER_SEL" gate="A" pin="2"/>
+<label x="33.02" y="190.5" size="1.27" layer="95" xref="yes"/>
+<wire x1="27.94" y1="190.5" x2="33.02" y2="190.5" width="0.1524" layer="91"/>
+</segment>
+<segment>
+<pinref part="C20" gate="G$1" pin="+"/>
+<wire x1="27.94" y1="162.56" x2="27.94" y2="165.1" width="0.1524" layer="91"/>
+<wire x1="27.94" y1="165.1" x2="27.94" y2="170.18" width="0.1524" layer="91"/>
+<wire x1="27.94" y1="170.18" x2="27.94" y2="175.26" width="0.1524" layer="91"/>
+<wire x1="27.94" y1="175.26" x2="30.48" y2="175.26" width="0.1524" layer="91"/>
+<label x="30.48" y="175.26" size="1.27" layer="95" xref="yes"/>
+<pinref part="L2" gate="G$1" pin="2"/>
+<wire x1="30.48" y1="170.18" x2="27.94" y2="170.18" width="0.1524" layer="91"/>
+<pinref part="L1" gate="G$1" pin="2"/>
+<wire x1="30.48" y1="165.1" x2="27.94" y2="165.1" width="0.1524" layer="91"/>
+</segment>
+</net>
+<net name="3V3PS" class="0">
+<segment>
+<pinref part="POWER_SEL" gate="A" pin="1"/>
+<wire x1="27.94" y1="187.96" x2="33.02" y2="187.96" width="0.1524" layer="91"/>
+<label x="33.02" y="187.96" size="1.27" layer="95" xref="yes"/>
+</segment>
+<segment>
+<pinref part="U$2" gate="G$1" pin="VOUT"/>
+<wire x1="15.24" y1="215.9" x2="15.24" y2="213.36" width="0.1524" layer="91"/>
+<label x="15.24" y="213.36" size="1.27" layer="95" xref="yes"/>
+</segment>
+</net>
+<net name="3V3ARDU" class="0">
+<segment>
+<pinref part="POWER_SEL" gate="A" pin="3"/>
+<wire x1="27.94" y1="193.04" x2="33.02" y2="193.04" width="0.1524" layer="91"/>
+<label x="33.02" y="193.04" size="1.27" layer="95" xref="yes"/>
+</segment>
 <segment>
 <pinref part="U2" gate="G$1" pin="3V"/>
@@
 </segment>
 </net>
-<net name="3V3IN" class="0">
-<segment>
-<pinref part="POWER_SEL" gate="A" pin="2"/>
-<label x="33.02" y="190.5" size="1.27" layer="95" xref="yes"/>
-<wire x1="27.94" y1="190.5" x2="33.02" y2="190.5" width="0.1524" layer="91"/>
-</segment>
-</net>
-<net name="3V3PS" class="0">
-<segment>
-<pinref part="POWER_SEL" gate="A" pin="1"/>
-<wire x1="27.94" y1="187.96" x2="33.02" y2="187.96" width="0.1524" layer="91"/>
-<label x="33.02" y="187.96" size="1.27" layer="95" xref="yes"/>
-</segment>
-</net>
-<net name="3V3ARDU" class="0">
-<segment>
-<pinref part="POWER_SEL" gate="A" pin="3"/>
-<wire x1="27.94" y1="193.04" x2="33.02" y2="193.04" width="0.1524" layer="91"/>
-<label x="33.02" y="193.04" size="1.27" layer="95" xref="yes"/>
-</segment>
-</net>
+<net name="PWRIN" class="0">
+<segment>
+<pinref part="J1" gate="G$1" pin="PWR"/>
+<wire x1="-73.66" y1="210.82" x2="-71.12" y2="210.82" width="0.1524" layer="91"/>
+<label x="-71.12" y="210.82" size="1.27" layer="95" xref="yes"/>
+</segment>
+<segment>
+<pinref part="U$2" gate="G$1" pin="VIN"/>
+<wire x1="-55.88" y1="215.9" x2="-58.42" y2="215.9" width="0.1524" layer="91"/>
+<label x="-58.42" y="215.9" size="1.27" layer="95" rot="R180" xref="yes"/>
+</segment>
+</net>
